File: hardware/winamp.kicad_pcb (KiCad board)
At the start: 2 copper layers, 2.1 x 1.7 mm, 13 parts, among them U101 TLV271QDBVRQ1, U102 ZXBM5210-SP

Commit message: WIP
Parts:
- added S3: TL1240GQ1JCLR, TL1240GQ1JCLR:SW_TL1240GQ1JCLR, F.Cu at (139.4, 104.3)
- added S4: TL1240GQ1JCLR, TL1240GQ1JCLR:SW_TL1240GQ1JCLR, F.Cu at (167.9, 104.2)
- added SW1: SW_Push, Buttons_Switches_THT:SW_PUSH_6mm_h7.3mm, F.Cu at (54.0, 101.8)
- added SW2: SW_Push, Buttons_Switches_THT:SW_PUSH_6mm_h7.3mm, F.Cu at (67.0, 101.8)
- added SW3: SW_Push, Buttons_Switches_THT:SW_PUSH_6mm_h7.3mm, F.Cu at (80.0, 101.8)
- added SW4: SW_Push, Buttons_Switches_THT:SW_PUSH_6mm_h7.3mm, F.Cu at (93.0, 101.8)
- added SW5: SW_Push, Buttons_Switches_THT:SW_PUSH_6mm_h7.3mm, F.Cu at (105.8, 101.8)
- added SW6: SW_Push, Buttons_Switches_THT:SW_PUSH_6mm_h7.3mm, F.Cu at (121.3, 101.8)
- added SW7: SW_Push, Buttons_Switches_THT:SW_PUSH_6mm_h7.3mm, F.Cu at (155.3, 102.0)
- moved C101 34.4 mm to (57.0, 88.8)
- moved R102 34.4 mm to (177.8, 97.6)
- moved R103 34.4 mm to (177.8, 84.6)
- moved U101 34.4 mm to (136.0, 94.8)
- moved C102 34.4 mm to (172.0, 97.4)
- moved C103 34.4 mm to (166.8, 97.2)
- moved U102 34.4 mm to (171.6, 90.2)

Commit message: alternative display test
Other:
- board text added: "MIPI 2.99 inch 268x800"
- board text added: "TFT IPS 4.58 inch ST7701S 320x960 SPI"
Changed lines of the file:
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@@
+  (gr_poly
+    (pts
+      (xy 98.153123 4.450265)
+      (xy 215.846878 4.450265)
+      (xy 215.846878 6.247327)
+      (xy 210.327821 6.247327)
+      (xy 100.22099 6.247327)
+      (xy 100.22099 42.953009)
+      (xy 210.327821 42.953009)
+      (xy 210.327821 6.247327)
+      (xy 215.846878 6.247327)
+      (xy 215.846878 44.749735)
+      (xy 98.153123 44.749735)
+    ) (layer "F.SilkS") (width 0.06655) (fill solid))
   (gr_poly
     (pts
@@
       (xy 97.8 81.194781)
     ) (layer "F.SilkS") (width 0.06655) (fill solid))
+  (gr_poly
+    (pts
+      (xy 98.29397 -23.236835)
+      (xy 176.90603 -23.236835)
+      (xy 176.90603 -20.343825)
+      (xy 171.423952 -20.343825)
+      (xy 171.421745 -20.431012)
+      (xy 171.415196 -20.517058)
+      (xy 171.404413 -20.601857)
+      (xy 171.3895 -20.685302)
+      (xy 171.370566 -20.767286)
+      (xy 171.347717 -20.847703)
+      (xy 171.32106 -20.926446)
+      (xy 171.290702 -21.003407)
+      (xy 171.256749 -21.078482)
+      (xy 171.219309 -21.151561)
+      (xy 171.178487 -21.22254)
+      (xy 171.134392 -21.291311)
+      (xy 171.087129 -21.357768)
+      (xy 171.036805 -21.421803)
+      (xy 170.983528 -21.483311)
+      (xy 170.927403 -21.542184)
+      (xy 170.868539 -21.598316)
+      (xy 170.807041 -21.6516)
+      (xy 170.743016 -21.701929)
+      (xy 170.676571 -21.749196)
+      (xy 170.607814 -21.793295)
+      (xy 170.53685 -21.83412)
+      (xy 170.463786 -21.871563)
+      (xy 170.38873 -21.905518)
+      (xy 170.311788 -21.935877)
+      (xy 170.233067 -21.962535)
+      (xy 170.152673 -21.985385)
+      (xy 170.070714 -22.004319)
+      (xy 169.987296 -22.019231)
+      (xy 169.902526 -22.030015)
+      (xy 169.81651 -22.036564)
+      (xy 169.729357 -22.03877)
+      (xy 101.244719 -22.03877)
+      (xy 101.157565 -22.036564)
+      (xy 101.071549 -22.030015)
+      (xy 100.986778 -22.019231)
+      (xy 100.903359 -22.004319)
+      (xy 100.821399 -21.985384)
+      (xy 100.741005 -21.962534)
+      (xy 100.662283 -21.935876)
+      (xy 100.585341 -21.905516)
+      (xy 100.510284 -21.871561)
+      (xy 100.437221 -21.834118)
+      (xy 100.366256 -21.793293)
+      (xy 100.297499 -21.749193)
+      (xy 100.231054 -21.701926)
+      (xy 100.167029 -21.651596)
+      (xy 100.105531 -21.598312)
+      (xy 100.046666 -21.54218)
+      (xy 99.990542 -21.483307)
+      (xy 99.937264 -21.421799)
+      (xy 99.886941 -21.357764)
+      (xy 99.839678 -21.291307)
+      (xy 99.795583 -21.222536)
+      (xy 99.754761 -21.151557)
+      (xy 99.717321 -21.078477)
+      (xy 99.683368 -21.003403)
+      (xy 99.65301 -20.926442)
+      (xy 99.626353 -20.847699)
+      (xy 99.603504 -20.767283)
+      (xy 99.58457 -20.685299)
+      (xy 99.569658 -20.601855)
+      (xy 99.558874 -20.517057)
+      (xy 99.552326 -20.431011)
+      (xy 99.550119 -20.343825)
+      (xy 99.550119 0.344191)
+      (xy 99.552326 0.431347)
+      (xy 99.558874 0.517366)
+      (xy 99.569658 0.602141)
+      (xy 99.58457 0.685566)
+      (xy 99.603504 0.767534)
+      (xy 99.626353 0.847937)
+      (xy 99.65301 0.926669)
+      (xy 99.683368 1.003624)
+      (xy 99.717321 1.078693)
+      (xy 99.754761 1.15177)
+      (xy 99.795583 1.222749)
+      (xy 99.839678 1.291521)
+      (xy 99.886941 1.357981)
+      (xy 99.937264 1.422022)
+      (xy 99.990542 1.483536)
+      (xy 100.046666 1.542417)
+      (xy 100.105531 1.598557)
+      (xy 100.167029 1.651851)
+      (xy 100.231054 1.70219)
+      (xy 100.297499 1.749468)
+      (xy 100.366256 1.793579)
+      (xy 100.437221 1.834415)
+      (xy 100.510284 1.871868)
+      (xy 100.585341 1.905834)
+      (xy 100.662283 1.936203)
+      (xy 100.741005 1.962871)
+      (xy 100.821399 1.985729)
+      (xy 100.903359 2.004671)
+      (xy 100.986778 2.019589)
+      (xy 101.071549 2.030377)
+      (xy 101.157565 2.036929)
+      (xy 101.244719 2.039137)
+      (xy 169.729357 2.039137)
+      (xy 169.816511 2.036929)
+      (xy 169.902527 2.030377)
+      (xy 169.987298 2.019589)
+      (xy 170.070717 2.00467)
+      (xy 170.152676 1.985728)
+      (xy 170.23307 1.96287)
+      (xy 170.311792 1.936202)
+      (xy 170.388734 1.905832)
+      (xy 170.463791 1.871867)
+      (xy 170.536854 1.834413)
+      (xy 170.607818 1.793577)
+      (xy 170.676576 1.749466)
+      (xy 170.74302 1.702187)
+      (xy 170.807045 1.651848)
+      (xy 170.868543 1.598554)
+      (xy 170.927407 1.542413)
+      (xy 170.983531 1.483532)
+      (xy 171.036808 1.422018)
+      (xy 171.087132 1.357977)
+      (xy 171.134394 1.291517)
+      (xy 171.17849 1.222744)
+      (xy 171.219311 1.151766)
+      (xy 171.256751 1.078688)
+      (xy 171.290704 1.003619)
+      (xy 171.321062 0.926665)
+      (xy 171.347718 0.847934)
+      (xy 171.370567 0.767531)
+      (xy 171.389501 0.685563)
+      (xy 171.404413 0.602139)
+      (xy 171.415197 0.517364)
+      (xy 171.421745 0.431346)
+      (xy 171.423952 0.344191)
+      (xy 171.423952 -20.343825)
+      (xy 176.90603 -20.343825)
+      (xy 176.90603 3.236835)
+      (xy 98.29397 3.236835)
+    ) (layer "F.SilkS") (width 0.06655) (fill solid))
+  (gr_text "MIPI 2.99 inch\n268x800" (at 136.6 -10) (layer "F.SilkS")
+    (effects (font (size 2.032 1.524) (thickness 0.3048)))
+  )
   (gr_text "OLED 3.12 inch green\nSSD1322\n256x64 SPI" (at 143.6 59.6) (layer "F.SilkS")
     (effects (font (size 2.032 1.524) (thickness 0.3048)))
@@
     (effects (font (size 2.032 1.524) (thickness 0.3048)))
   )
+  (gr_text "TFT IPS 4.58 inch\nST7701S\n320x960 SPI" (at 158.4 24.8) (layer "F.SilkS")
+    (effects (font (size 2.032 1.524) (thickness 0.3048)))
+  )
+  (group "" (id 24868189-6c76-4bfa-a404-5bd24ac5e82f)
+    (members
+      70410037-ee39-4007-aa32-79cb7fcbe65e
+    )
+  )
   (group "" (id 30ead398-6d63-45e0-93e9-14f385270c33)
     (members
@@
     )
   )
+  (group "" (id 63a54e1c-6a5d-4a95-adce-c0db36ea7f25)
+    (members
+      4e4a1bbe-32ba-4e9d-9824-341ca54ce26a
+    )
+  )
