File: hardware/winamp.kicad_sch (KiCad schematic)
At the start: 13 parts, among them U101 TLV271QDBVRQ1, U102 ZXBM5210-SP

Commit message: WIP
Parts:
- added S3, S4: TL1240GQ1JCLR, TL1240GQ1JCLR:SW_TL1240GQ1JCLR, symbol TL1240GQ1JCLR:TL1240GQ1JCLR
- added SW1, SW3, SW4, SW5, SW6, SW7: SW_Push, symbol Switch:SW_Push
- added SW2: (no value), symbol Switch:SW_Push
Changed lines of the file:
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@@
     (pin "T")
+  )
+  (symbol (lib_id "TL1240GQ1JCLR:TL1240GQ1JCLR") (at 86.36 191.77 0) (unit 1)
+    (in_bom yes) (on_board yes) (fields_autoplaced)
+    (property "Reference" "S3" (id 0) (at 86.36 179.07 0))
+    (property "Value" "TL1240GQ1JCLR" (id 1) (at 86.36 181.61 0))
+    (property "Footprint" "TL1240GQ1JCLR:SW_TL1240GQ1JCLR" (id 2) (at 86.36 191.77 0)
+      (effects (font (size 1.27 1.27)) (justify bottom) hide)
+    )
+    (property "Datasheet" "" (id 3) (at 86.36 191.77 0)
+      (effects (font (size 1.27 1.27)) hide)
+    )
+    (property "MANUFACTURER" "E-Switch" (id 4) (at 86.36 191.77 0)
+      (effects (font (size 1.27 1.27)) (justify bottom) hide)
+    )
+    (property "PARTREV" "B" (id 5) (at 86.36 191.77 0)
+      (effects (font (size 1.27 1.27)) (justify bottom) hide)
+    )
+    (property "STANDARD" "Manufacturer Recommendations" (id 6) (at 86.36 191.77 0)
+      (effects (font (size 1.27 1.27)) (justify bottom) hide)
+    )
+    (property "MAXIMUM_PACKAGE_HEIGHT" "7.18.2022" (id 7) (at 86.36 191.77 0)
+      (effects (font (size 1.27 1.27)) (justify bottom) hide)
+    )
+    (property "SNAPEDA_PN" "TL1240GQ1JCLR" (id 8) (at 86.36 191.77 0)
+      (effects (font (size 1.27 1.27)) (justify bottom) hide)
+    )
+    (pin "+")
+    (pin "-")
+    (pin "1")
+    (pin "2")
+    (pin "3")
+    (pin "4")
+  )
+  (symbol (lib_id "Switch:SW_Push") (at 59.69 167.64 0) (unit 1)
+    (in_bom yes) (on_board yes) (fields_autoplaced)
+    (property "Reference" "SW6" (id 0) (at 59.69 160.02 0))
+    (property "Value" "SW_Push" (id 1) (at 59.69 162.56 0))
+    (property "Footprint" "" (id 2) (at 59.69 162.56 0)
+      (effects (font (size 1.27 1.27)) hide)
+    )
+    (property "Datasheet" "~" (id 3) (at 59.69 162.56 0)
+      (effects (font (size 1.27 1.27)) hide)
+    )
+    (pin "1")
+    (pin "2")
   )
   (symbol (lib_id "Device:R") (at 102.87 64.77 90) (unit 1)
@@
     )
     (property "Datasheet" "~" (id 3) (at 132.08 34.29 0)
+      (effects (font (size 1.27 1.27)) hide)
+    )
+    (pin "1")
+    (pin "2")
+  )
+  (symbol (lib_id "Switch:SW_Push") (at 48.26 195.58 0) (unit 1)
+    (in_bom yes) (on_board yes) (fields_autoplaced)
+    (property "Reference" "SW5" (id 0) (at 48.26 187.96 0))
+    (property "Value" "SW_Push" (id 1) (at 48.26 190.5 0))
+    (property "Footprint" "" (id 2) (at 48.26 190.5 0)
+      (effects (font (size 1.27 1.27)) hide)
+    )
+    (property "Datasheet" "~" (id 3) (at 48.26 190.5 0)
+      (effects (font (size 1.27 1.27)) hide)
+    )
+    (pin "1")
+    (pin "2")
+  )
+  (symbol (lib_id "Switch:SW_Push") (at 27.94 182.88 0) (unit 1)
+    (in_bom yes) (on_board yes) (fields_autoplaced)
+    (property "Reference" "SW1" (id 0) (at 27.94 175.26 0))
+    (property "Value" "SW_Push" (id 1) (at 27.94 177.8 0))
+    (property "Footprint" "" (id 2) (at 27.94 177.8 0)
+      (effects (font (size 1.27 1.27)) hide)
+    )
+    (property "Datasheet" "~" (id 3) (at 27.94 177.8 0)
+      (effects (font (size 1.27 1.27)) hide)
+    )
+    (pin "1")
+    (pin "2")
+  )
+  (symbol (lib_id "Switch:SW_Push") (at 44.45 180.34 0) (unit 1)
+    (in_bom yes) (on_board yes) (fields_autoplaced)
+    (property "Reference" "SW4" (id 0) (at 44.45 172.72 0))
+    (property "Value" "SW_Push" (id 1) (at 44.45 175.26 0))
+    (property "Footprint" "" (id 2) (at 44.45 175.26 0)
+      (effects (font (size 1.27 1.27)) hide)
+    )
+    (property "Datasheet" "~" (id 3) (at 44.45 175.26 0)
+      (effects (font (size 1.27 1.27)) hide)
+    )
+    (pin "1")
+    (pin "2")
+  )
+  (symbol (lib_id "TL1240GQ1JCLR:TL1240GQ1JCLR") (at 113.03 190.5 0) (unit 1)
+    (in_bom yes) (on_board yes) (fields_autoplaced)
+    (property "Reference" "S4" (id 0) (at 113.03 177.8 0))
+    (property "Value" "TL1240GQ1JCLR" (id 1) (at 113.03 180.34 0))
+    (property "Footprint" "TL1240GQ1JCLR:SW_TL1240GQ1JCLR" (id 2) (at 113.03 190.5 0)
+      (effects (font (size 1.27 1.27)) (justify bottom) hide)
+    )
+    (property "Datasheet" "" (id 3) (at 113.03 190.5 0)
+      (effects (font (size 1.27 1.27)) hide)
+    )
+    (property "MANUFACTURER" "E-Switch" (id 4) (at 113.03 190.5 0)
+      (effects (font (size 1.27 1.27)) (justify bottom) hide)
+    )
+    (property "PARTREV" "B" (id 5) (at 113.03 190.5 0)
+      (effects (font (size 1.27 1.27)) (justify bottom) hide)
+    )
+    (property "STANDARD" "Manufacturer Recommendations" (id 6) (at 113.03 190.5 0)
+      (effects (font (size 1.27 1.27)) (justify bottom) hide)
+    )
+    (property "MAXIMUM_PACKAGE_HEIGHT" "7.18.2022" (id 7) (at 113.03 190.5 0)
+      (effects (font (size 1.27 1.27)) (justify bottom) hide)
+    )
+    (property "SNAPEDA_PN" "TL1240GQ1JCLR" (id 8) (at 113.03 190.5 0)
+      (effects (font (size 1.27 1.27)) (justify bottom) hide)
+    )
+    (pin "+")
+    (pin "-")
+    (pin "1")
+    (pin "2")
+    (pin "3")
+    (pin "4")
+  )
+  (symbol (lib_id "Switch:SW_Push") (at 43.18 167.64 0) (unit 1)
+    (in_bom yes) (on_board yes) (fields_autoplaced)
+    (property "Reference" "SW3" (id 0) (at 43.18 160.02 0))
+    (property "Value" "SW_Push" (id 1) (at 43.18 162.56 0))
+    (property "Footprint" "" (id 2) (at 43.18 162.56 0)
+      (effects (font (size 1.27 1.27)) hide)
+    )
+    (property "Datasheet" "~" (id 3) (at 43.18 162.56 0)
       (effects (font (size 1.27 1.27)) hide)
     )
@@
     (pin "9")
   )
+  (symbol (lib_id "Switch:SW_Push") (at 30.48 168.91 0) (unit 1)
+    (in_bom yes) (on_board yes) (fields_autoplaced)
+    (property "Reference" "SW2" (id 0) (at 30.48 161.29 0))
+    (property "Value" "" (id 1) (at 30.48 163.83 0))
+    (property "Footprint" "" (id 2) (at 30.48 163.83 0)
+      (effects (font (size 1.27 1.27)) hide)
+    )
+    (property "Datasheet" "~" (id 3) (at 30.48 163.83 0)
+      (effects (font (size 1.27 1.27)) hide)
+    )
+    (pin "1")
+    (pin "2")
+  )
+  (symbol (lib_id "Switch:SW_Push") (at 63.5 181.61 0) (unit 1)
+    (in_bom yes) (on_board yes) (fields_autoplaced)
+    (property "Reference" "SW7" (id 0) (at 63.5 173.99 0))
+    (property "Value" "SW_Push" (id 1) (at 63.5 176.53 0))
+    (property "Footprint" "" (id 2) (at 63.5 176.53 0)
+      (effects (font (size 1.27 1.27)) hide)
+    )
+    (property "Datasheet" "~" (id 3) (at 63.5 176.53 0)
+      (effects (font (size 1.27 1.27)) hide)
+    )
+    (pin "1")
+    (pin "2")
+  )
   (symbol (lib_id "Device:C") (at 146.05 40.64 90) (unit 1)
     (in_bom yes) (on_board yes) (fields_autoplaced)
@@
       (reference "S2") (unit 1) (value "TL1240GQ1JCLR") (footprint "TL1240GQ1JCLR:SW_TL1240GQ1JCLR")
     )
+    (path "/24e7742a-9d34-4aba-8d0f-ac7f019e8fa2"
+      (reference "S3") (unit 1) (value "TL1240GQ1JCLR") (footprint "TL1240GQ1JCLR:SW_TL1240GQ1JCLR")
+    )
+    (path "/787c60d8-b7db-443b-a24a-37f0e937d105"
+      (reference "S4") (unit 1) (value "TL1240GQ1JCLR") (footprint "TL1240GQ1JCLR:SW_TL1240GQ1JCLR")
+    )
+    (path "/5995dc43-9510-4a55-a4df-221a8a7f6678"
+      (reference "SW1") (unit 1) (value "SW_Push") (footprint "Buttons_Switches_THT:SW_PUSH_6mm_h7.3mm")
+    )
+    (path "/a8836da4-9984-4d9f-bc1c-845122baea3f"
+      (reference "SW2") (unit 1) (value "SW_Push") (footprint "Buttons_Switches_THT:SW_PUSH_6mm_h7.3mm")
+    )
+    (path "/80674178-0b08-4edb-a33a-fc02015562f5"
+      (reference "SW3") (unit 1) (value "SW_Push") (footprint "Buttons_Switches_THT:SW_PUSH_6mm_h7.3mm")
+    )
+    (path "/69acca36-ed08-40ef-aeab-898d13c7e746"
+      (reference "SW4") (unit 1) (value "SW_Push") (footprint "Buttons_Switches_THT:SW_PUSH_6mm_h7.3mm")
+    )
+    (path "/45453541-2927-4c40-885b-89c0b8de52d8"
+      (reference "SW5") (unit 1) (value "SW_Push") (footprint "Buttons_Switches_THT:SW_PUSH_6mm_h7.3mm")
+    )
+    (path "/297a413b-8372-49d7-a3cc-b20b59ff6c53"
+      (reference "SW6") (unit 1) (value "SW_Push") (footprint "Buttons_Switches_THT:SW_PUSH_6mm_h7.3mm")
+    )
+    (path "/ac90e65b-ad5d-4521-84ea-fe9f17bdf3da"
+      (reference "SW7") (unit 1) (value "SW_Push") (footprint "Buttons_Switches_THT:SW_PUSH_6mm_h7.3mm")
+    )
     (path "/b9e7c4bd-a5c2-45f2-a58f-82ef10914d37"
